File: Hardware/CoreLogger.sch (EAGLE design)
At the start: 32 parts, among them J1 CONN_32.54_SCREW, J2 CONN_32.54_SCREW, J4 CONN_5, J6 CONN_42.54, J7 CONN_42.54, J8 CONN_42.54, Q1 DMG3404, U1 TPS62200SOT23, U2 SN74AUP1G34SC70, U3 MIC2544MSOP, U4 MIC2544MSOP

Commit message: Added Eagle library, continued logger designs
Parts:
- added BT1: BATTERY_COIN12MM, bschulz:BATTERY_COIN12MM
- added C10: 0.1uF, bschulz_passives:C-EU0.1UFC0603
- added C9: (no value), bschulz_passives:C-EUC0603
- added J10: CONN_42.54_SCREW, bschulz:CONN_42.54_SCREW
- added J11, J12: CONN_32.54_SCREW, bschulz:CONN_32.54_SCREW
- added JP1: JUMPER-SMT_2_NO_SILK, SparkFun-Jumpers:JUMPER-SMT_2_NO_SILK
- added R10, R11: 10M, bschulz_passives:R-EU_10MR0603
- added R12: 100m, bschulz_passives:R-EU_R0805
- added R41: 10k, bschulz_passives:R-EU_10KR0402
- added R7, R8: (no value), bschulz_passives:R-EU_R0603
- added R9: 10m, bschulz_passives:R-EU_R0805
- added RTC1: DS3231M, bschulz:DS3231M
- added SD1: MICROSDCD, bschulz:MICROSDCD
- added U$1: POLOLU_REGULATOR, LEAF_Components:POLOLU_REGULATOR
- added U10: (no value), bschulz:SN74AUP1G14DCK
- added U11: MCP23018QFN, bschulz:MCP23018QFN
- added U12: TLV3691DCK, bschulz:TLV3691DCK
- added U13, U14: INA219DCN, bschulz:INA219DCN
- added U5: LTC2054, bschulz:LTC2054
- added U6, U7: (no value), bschulz:SN74HC590AD
- added U8, U9: (no value), bschulz:SN74HC165D
- added XU1: MAX31856_BREAKOUT, LEAF_Components:MAX31856_BREAKOUT
- J6, J7, J8: value CONN_42.54 -> CONN_42.54_SCREW; device bschulz:CONN_42.54 -> bschulz:CONN_42.54_SCREW
- MS1: value FEATHERWING -> FEATHERWING_NODIM; device adafruit:FEATHERWING -> adafruit:FEATHERWING_NODIM
Connections:
- removed net SAP_THERM: J6.4
- new net !LOAD: U10G1.Y, U6.RCLK, U7.RCLK
- new net !RESET: MS1.!RESET, U11.!RESET
- new net !RST: U6.!CCLR, U7.!CCLR
- new net CLK: MS1.GPIO13, U8.CLK, U9.CLK
- new net DATA: MS1.GPIO12, U9.QH
- new net INTA: MS1.GPIO6, U11.INTA
- new net LOAD: U10G1.A, U8.SH/!LD, U9.SH/!LD
- new net MISO: MS1.GPIOMISO, SD1.DATA_OUT, XU1.SDO
- new net MOSI: MS1.GPIOMOSI, SD1.DATA_IN, XU1.SDI
- new net N$10: U7.QD, U9.D
- new net N$11: U7.QE, U9.E
- new net N$12: U7.QF, U9.F
- new net N$13: U7.QG, U9.G
- new net N$14: U7.QH, U9.H
- new net N$15: U6.QH, U8.H
- new net N$16: U6.QG, U8.G
- new net N$17: U6.QF, U8.F
- new net N$18: U6.QE, U8.E
- new net N$19: U6.QD, U8.D
- new net N$2: C9.1, R8.2, U5.VIN-
- new net N$20: U6.QC, U8.C
- new net N$21: U6.QB, U8.B
- new net N$22: U6.QA, U8.A
- new net N$23: U8.QH, U9.SER
- new net N$24: U6.!RCO, U7.CCLK
- new net N$26: U11.INTB
- new net N$30: BT1.+, C10.1, RTC1.VBAT
- new net N$7: U7.QA, U9.A
- new net N$8: U7.QB, U9.B
- new net N$9: U7.QC, U9.C
- new net PULSE_DIG: U12.OUT, U6.CCLK
- new net PYRO_AMP: C9.2, JP1.2, MS1.GPIOA0, R7.2, U5.OUT
- new net SAP_CS: MS1.GPIOA5, XU1.CS
- new net SAP_FAULT: XU1.FLT
- new net SAP_READY: XU1.DRDY
- new net SAP_THERM+: J6.3, XU1.THERM+
- new net SAP_THERM-: J6.4, XU1.THERM-
- new net SCK: MS1.GPIOSCK, SD1.SCLK, XU1.SCK
- new net SD_CD: R41.1, SD1.CARD_DETECT
- new net SD_CS: MS1.GPIO10, SD1.CS
- new net SOIL_1: J11.2, MS1.GPIOA3
- new net SOIL_2: J12.2, MS1.GPIOA2
- new net VBAT: J10.2, R12.2, R9.1, U13.VIN-, U14.VIN+
- new net VCC: U6.VCC, U7.VCC, U8.VCC, U9.VCC
- new net VMAIN: R12.1, U$1.VIN, U14.VIN-
- new net VREF: R10.1, R11.1, U12.IN-
- new net VSOLAR: J10.4, R9.2, U13.VIN+
- new net V_CAP: R10.2
- net 3V3: now also R41.2, RTC1.VCC, SD1.VDD, U11.VDD, U13.VSS, U14.A0, U14.VSS
- net 3V3_AUX: now also J11.3, J12.3, U10G2.P$V+, U12.VCC, U5.VDD
- net 5V: now also U$1.VOUT
- net 5V_AUX: now also XU1.VIN
- net F_IN: now also MS1.GPIO11
- net GND: now also BT1.-, C10.2, J10.1, J10.3, J11.1, J12.1, R11.2, RTC1.GND, SD1.CARD_DETECT1, SD1.GND, SD1.GND1, SD1.VSS, U$1.GND, U10G2.P$V-, U11.ADDR, U11.VSS, U12.GND, U13.A0, U13.A1, U13.GND, U14.A1, U14.GND, U5.VIN+, U5.VSS, U6.!CCKEN, U6.!OE, U6.GND, U7.!CCKEN, U7.!OE, U7.GND, U8.CLK_INH, U8.GND, U8.SER, U9.CLK_INH, U9.GND, XU1.GND; no longer J6.3
- net PYRO: now also JP1.1, R7.1, R8.1
- net RAIN_TIP: now also MS1.GPIO9
- net SCL: now also RTC1.SCL, U11.SCL, U13.SCL, U14.SCL
- net SDA: now also RTC1.SDA, U11.SDA, U13.SDA, U14.SDA
- net WATER_DEPTH_3V3: now also MS1.GPIOA1
- net WATER_TEMP: now also MS1.GPIO5
- net WIND_PULSE: now also U12.IN+
Other:
- note added: "Add alternative amp structure?"
- note added: "Add test points!"
- note added: "Check addresses"
- note added: "Connect to Paticle!"
- note added: "Connect to Paticle?"
- note added: "Connect: Clk DATA SDA SCL RAIN_TIP PYRO_AMP? WATER_DEPTH_3V3 WATER_TEMP MOSI MISO SCK CS_SAP SAP_HEATER_SW INTA INTB F_IN"
- note added: "Connect: LOAD RST S0 S1 5v_FAULT 3v3_FAULT 3v3_EN 5v_EN HEATER_EN SAP_FAULT SAP_READY SD_CD"
- note added: "Pullup for input pulse line"
- note added: "Replace with real molex!"
- note removed: "Add IO expander"
- note removed: "Add SD card? Add RTC?"

Commit message: Routing and minor design updates
The majority of functionality is present, passes DRC, need to add polygons and test points, along with labeling
Parts:
- added C11: 0.1uF, bschulz_passives:C-EU0.1UFC0402
- added F1: PPTC100MA1210, bschulz:PPTC100MA1210
- added H1, H2, H3: (no value), bschulz:MOUNTING_HOLE4_NP
- added R13: 10k, bschulz_passives:R-EU_10KR0603
Connections:
- removed net 3V3_EN: U4.EN
- removed net 5V_EN: U3.EN
- removed net VCC: U6.VCC, U7.VCC, U8.VCC, U9.VCC
- removed net V_CAP: R10.2
- new net 3V3_WIND: F1.2, J9.2
- new net AUX_EN: U11.GPA1, U3.EN, U4.EN
- net !RST: now also U11.GPB6
- net 3V3: now also F1.1, R10.2, U10G2.P$V+, U12.VCC, U6.VCC, U7.VCC, U8.VCC, U9.VCC
- net 3V3_AUX: now also C11.1, R13.2; no longer J9.2, U10G2.P$V+, U12.VCC
- net 3V3_FAULT: now also U11.GPA0
- net 5V_FAULT: now also U11.GPA2
- net GND: now also C11.2
- net HEATER_EN: now also U11.GPA3
- net LOAD: now also U11.GPB7
- net S0: now also U11.GPB1
- net S1: now also U11.GPB2
- net SAP_FAULT: now also U11.GPB4
- net SAP_HEATER_SW: now also MS1.GPIOA4
- net SAP_READY: now also U11.GPB3
- net SD_CD: now also U11.GPB5
- net SOIL_1: now also J12.2; no longer J11.2
- net SOIL_2: now also J11.2; no longer J12.2
- net WATER_TEMP: now also R13.1
Other:
- note added: "Add caps???"
- note added: "Add test points!!"
- note added: "Remove??"

Commit message: Further updates, ready for final review
Added silkscreen and minor layout improvements
Parts:
- added C12, C13, C14, C15, C16, C17: 0.1uF, bschulz_passives:C-EU0.1UFC0402
- added H4, H5: (no value), bschulz:MOUNTING_HOLE4_NP
Connections:
- net 3V3: now also C12.1, C13.1, C14.1, C15.1, C16.1, C17.1
- net GND: now also C12.2, C13.2, C14.2, C15.2, C16.2, C17.2
Changed lines of the file:
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@@
 <setting verticaltext="up"/>
 </settings>
-<grid distance="0.1" unitdist="inch" unit="mm" style="lines" multiple="1" display="yes" altdistance="0.01" altunitdist="inch" altunit="inch"/>
+<grid distance="0.1" unitdist="inch" unit="mm" style="lines" multiple="1" display="no" altdistance="0.01" altunitdist="inch" altunit="inch"/>
 <layers>
 <layer number="1" name="Top" color="4" fill="1" visible="yes" active="no"/>
@@
 <part name="GND29" library="supply1" library_urn="urn:adsk.eagle:library:371" deviceset="GND" device=""/>
 <part name="F1" library="bschulz" deviceset="PPTC" device="1210" technology="100MA" value="PPTC100MA1210"/>
+<part name="C12" library="bschulz_passives" deviceset="C-EU" device="C0402" technology="0.1UF" value="0.1uF"/>
+<part name="C13" library="bschulz_passives" deviceset="C-EU" device="C0402" technology="0.1UF" value="0.1uF"/>
+<part name="GND30" library="supply1" library_urn="urn:adsk.eagle:library:371" deviceset="GND" device=""/>
+<part name="GND31" library="supply1" library_urn="urn:adsk.eagle:library:371" deviceset="GND" device=""/>
+<part name="C14" library="bschulz_passives" deviceset="C-EU" device="C0402" technology="0.1UF" value="0.1uF"/>
+<part name="GND32" library="supply1" library_urn="urn:adsk.eagle:library:371" deviceset="GND" device=""/>
+<part name="C15" library="bschulz_passives" deviceset="C-EU" device="C0402" technology="0.1UF" value="0.1uF"/>
+<part name="GND33" library="supply1" library_urn="urn:adsk.eagle:library:371" deviceset="GND" device=""/>
+<part name="C16" library="bschulz_passives" deviceset="C-EU" device="C0402" technology="0.1UF" value="0.1uF"/>
+<part name="GND34" library="supply1" library_urn="urn:adsk.eagle:library:371" deviceset="GND" device=""/>
+<part name="C17" library="bschulz_passives" deviceset="C-EU" device="C0402" technology="0.1UF" value="0.1uF"/>
+<part name="GND35" library="supply1" library_urn="urn:adsk.eagle:library:371" deviceset="GND" device=""/>
+<part name="H4" library="bschulz" deviceset="MOUNTING_HOLE" device="4_NP"/>
+<part name="H5" library="bschulz" deviceset="MOUNTING_HOLE" device="4_NP"/>
 </parts>
 <sheets>
@@
 <attribute name="VALUE" x="397.51" y="256.286" size="1.778" layer="96" font="vector" align="top-center"/>
 </instance>
+<instance part="C12" gate="G$1" x="81.28" y="180.34" smashed="yes">
+<attribute name="NAME" x="82.804" y="180.721" size="1.778" layer="95"/>
+<attribute name="VALUE" x="82.804" y="175.641" size="1.778" layer="96"/>
+</instance>
+<instance part="C13" gate="G$1" x="81.28" y="205.74" smashed="yes">
+<attribute name="NAME" x="82.804" y="206.121" size="1.778" layer="95"/>
+<attribute name="VALUE" x="82.804" y="201.041" size="1.778" layer="96"/>
+</instance>
+<instance part="GND30" gate="1" x="81.28" y="170.18" smashed="yes">
+<attribute name="VALUE" x="78.74" y="167.64" size="1.778" layer="96"/>
+</instance>
+<instance part="GND31" gate="1" x="81.28" y="195.58" smashed="yes">
+<attribute name="VALUE" x="78.74" y="193.04" size="1.778" layer="96"/>
+</instance>
+<instance part="C14" gate="G$1" x="276.86" y="134.62" smashed="yes">
+<attribute name="NAME" x="278.384" y="135.001" size="1.778" layer="95"/>
+<attribute name="VALUE" x="278.384" y="129.921" size="1.778" layer="96"/>
+</instance>
+<instance part="GND32" gate="1" x="276.86" y="124.46" smashed="yes">
+<attribute name="VALUE" x="274.32" y="121.92" size="1.778" layer="96"/>
+</instance>
+<instance part="C15" gate="G$1" x="15.24" y="287.02" smashed="yes">
+<attribute name="NAME" x="16.764" y="287.401" size="1.778" layer="95"/>
+<attribute name="VALUE" x="16.764" y="282.321" size="1.778" layer="96"/>
+</instance>
+<instance part="GND33" gate="1" x="15.24" y="276.86" smashed="yes">
+<attribute name="VALUE" x="12.7" y="274.32" size="1.778" layer="96"/>
+</instance>
+<instance part="C16" gate="G$1" x="236.22" y="281.94" smashed="yes">
+<attribute name="NAME" x="237.744" y="282.321" size="1.778" layer="95"/>
+<attribute name="VALUE" x="237.744" y="277.241" size="1.778" layer="96"/>
+</instance>
+<instance part="GND34" gate="1" x="236.22" y="271.78" smashed="yes">
+<attribute name="VALUE" x="233.68" y="269.24" size="1.778" layer="96"/>
+</instance>
+<instance part="C17" gate="G$1" x="81.28" y="40.64" smashed="yes">
+<attribute name="NAME" x="82.804" y="41.021" size="1.778" layer="95"/>
+<attribute name="VALUE" x="82.804" y="35.941" size="1.778" layer="96"/>
+</instance>
+<instance part="GND35" gate="1" x="81.28" y="30.48" smashed="yes">
+<attribute name="VALUE" x="78.74" y="27.94" size="1.778" layer="96"/>
+</instance>
 </instances>
 <busses>
@@
 <pinref part="GND29" gate="1" pin="GND"/>
 </segment>
+<segment>
+<pinref part="C12" gate="G$1" pin="2"/>
+<wire x1="81.28" y1="175.26" x2="81.28" y2="172.72" width="0.1524" layer="91"/>
+<pinref part="GND30" gate="1" pin="GND"/>
+</segment>
+<segment>
+<pinref part="C13" gate="G$1" pin="2"/>
+<wire x1="81.28" y1="200.66" x2="81.28" y2="198.12" width="0.1524" layer="91"/>
+<pinref part="GND31" gate="1" pin="GND"/>
+</segment>
+<segment>
+<pinref part="C14" gate="G$1" pin="2"/>
+<wire x1="276.86" y1="129.54" x2="276.86" y2="127" width="0.1524" layer="91"/>
+<pinref part="GND32" gate="1" pin="GND"/>
+</segment>
+<segment>
+<pinref part="C15" gate="G$1" pin="2"/>
+<wire x1="15.24" y1="281.94" x2="15.24" y2="279.4" width="0.1524" layer="91"/>
+<pinref part="GND33" gate="1" pin="GND"/>
+</segment>
+<segment>
+<pinref part="C16" gate="G$1" pin="2"/>
+<wire x1="236.22" y1="276.86" x2="236.22" y2="274.32" width="0.1524" layer="91"/>
+<pinref part="GND34" gate="1" pin="GND"/>
+</segment>
+<segment>
+<pinref part="C17" gate="G$1" pin="2"/>
+<wire x1="81.28" y1="35.56" x2="81.28" y2="33.02" width="0.1524" layer="91"/>
+<pinref part="GND35" gate="1" pin="GND"/>
+</segment>
 </net>
 <net name="WIND_PULSE" class="0">
@@
 <pinref part="R10" gate="G$1" pin="2"/>
 <pinref part="P+1" gate="VCC" pin="VCC"/>
+</segment>
+<segment>
+<pinref part="C12" gate="G$1" pin="1"/>
+<wire x1="81.28" y1="182.88" x2="81.28" y2="185.42" width="0.1524" layer="91"/>
+<wire x1="81.28" y1="185.42" x2="83.82" y2="185.42" width="0.1524" layer="91"/>
+<label x="83.82" y="185.42" size="1.778" layer="95" xref="yes"/>
+</segment>
+<segment>
+<pinref part="C13" gate="G$1" pin="1"/>
+<wire x1="81.28" y1="208.28" x2="81.28" y2="210.82" width="0.1524" layer="91"/>
+<wire x1="81.28" y1="210.82" x2="83.82" y2="210.82" width="0.1524" layer="91"/>
+<label x="83.82" y="210.82" size="1.778" layer="95" xref="yes"/>
+</segment>
+<segment>
+<pinref part="C14" gate="G$1" pin="1"/>
+<wire x1="276.86" y1="137.16" x2="276.86" y2="139.7" width="0.1524" layer="91"/>
+<wire x1="276.86" y1="139.7" x2="279.4" y2="139.7" width="0.1524" layer="91"/>
+<label x="279.4" y="139.7" size="1.778" layer="95" xref="yes"/>
+</segment>
+<segment>
+<pinref part="C15" gate="G$1" pin="1"/>
+<wire x1="15.24" y1="289.56" x2="15.24" y2="292.1" width="0.1524" layer="91"/>
+<wire x1="15.24" y1="292.1" x2="17.78" y2="292.1" width="0.1524" layer="91"/>
+<label x="17.78" y="292.1" size="1.778" layer="95" xref="yes"/>
+</segment>
+<segment>
+<pinref part="C16" gate="G$1" pin="1"/>
+<wire x1="236.22" y1="284.48" x2="236.22" y2="287.02" width="0.1524" layer="91"/>
+<wire x1="236.22" y1="287.02" x2="238.76" y2="287.02" width="0.1524" layer="91"/>
+<label x="238.76" y="287.02" size="1.778" layer="95" xref="yes"/>
+</segment>
+<segment>
+<pinref part="C17" gate="G$1" pin="1"/>
+<wire x1="81.28" y1="43.18" x2="81.28" y2="45.72" width="0.1524" layer="91"/>
+<wire x1="81.28" y1="45.72" x2="83.82" y2="45.72" width="0.1524" layer="91"/>
+<label x="83.82" y="45.72" size="1.778" layer="95" xref="yes"/>
 </segment>
 </net>
@@
 <attribute name="VALUE" x="103.632" y="109.2962" size="1.778" layer="96"/>
 </instance>
+<instance part="H4" gate="G$1" x="111.76" y="111.76" smashed="yes">
+<attribute name="NAME" x="113.792" y="112.3442" size="1.778" layer="95"/>
+<attribute name="VALUE" x="113.792" y="109.2962" size="1.778" layer="96"/>
+</instance>
+<instance part="H5" gate="G$1" x="119.38" y="111.76" smashed="yes">
+<attribute name="NAME" x="121.412" y="112.3442" size="1.778" layer="95"/>
+<attribute name="VALUE" x="121.412" y="109.2962" size="1.778" layer="96"/>
+</instance>
 </instances>
