File: Hardware/CoreLogger_TopLoadMicro_CD.brd (EAGLE design)
At the start: 80 x 80 mm, 75 parts, among them J1 CONN_32.54_SCREW, J10 CONN_42.54_SCREW, J11 CONN_32.54_SCREW, J12 CONN_32.54_SCREW, J13 CONN_62.54, J2 CONN_32.54_SCREW, J4 CONN_5, J6 CONN_42.54_SCREW, J7 CONN_42.54_SCREW, J8 CONN_42.54_SCREW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

Commit message: Generated optional board designs, generated gerbers
Parts:
- SD1: value MICROSDCD -> MICROSDHINDGED; device bschulz:MICROSD_CD -> bschulz:MICROSD_HIROSE_HINDGED
- moved SD1 7.68 mm to (2.86, 43.8), turned to 270 degrees
Connections:
- net GND: no longer SD1.CD2
- net SD_CD: now also SD1.CD; no longer SD1.CD1
Routing:
- net MISO: track 69.8 -> 73.6 mm
- net SCK: track 56.1 -> 59.0 mm
- net GND: track 602.6 -> 605.5 mm
- net 3V3: track 283.1 -> 285.5 mm
- net SD_CS: track 63.6 -> 65.8 mm
- net MOSI: track 61.8 -> 64.1 mm
- net SD_CD: track 19.7 -> 20.9 mm
- net PULSE_DIG: track 42.5 -> 43.4 mm
